File: 3D4E Macropad.kicad_sch (KiCad schematic)
At the start: 20 parts, among them U1 Pico, U2 KY-040

Commit message: macropad update final
Parts:
- removed D1, D2, D3, D4, D5, D6, D7, D8, D9: D_Small, Diode_SMD:D_SOD-123, symbol Device:D_Small
- added D1, D10, D2, D3, D4, D5, D6, D7, D8: 1N4148, 1N4148-Diode:DIOAD829W49L456D191, symbol 1N4148:1N4148
- added ssd1: 3, KiCad-SSD1306-0.91-OLED-4pin-128x32.pretty-master:SSD1306-0.91-OLED-4pin-128x32, symbol ssd1306:ssd1306_0.91
Connections:
- net Col 0: now also U1.9 (GPIO6); no longer U1.6 (GPIO4)
- net Col 1: now also U1.10 (GPIO7); no longer U1.5 (GPIO3)
- net Col 2: now also U1.11 (GPIO8); no longer U1.4 (GPIO2)
- net GND: now also U1.13 (GND), U1.18 (GND), U1.8 (GND), ssd1.1 (GND)
- net KY040-CLK: now also U1.1 (GPIO0); no longer U1.31 (GPIO26_ADC0)
- net KY040-DT: now also U1.2 (GPIO1); no longer U1.32 (GPIO27_ADC1)
- net KY040-SW: now also U1.4 (GPIO2); no longer U1.34 (GPIO28_ADC2)
- net Row_0: now also U1.17 (GPIO13), D1.C, D10.C, D2.C; no longer U1.12 (GPIO9)
- net Row_1: now also U1.19 (GPIO14), D3.C, D4.C, D5.C; no longer U1.13 (GND)
- net Row_2: now also U1.20 (GPIO15), D6.C, D7.C, D8.C; no longer U1.29 (GPIO22)
- net SSD1306-SCK: now also U1.7 (GPIO5), ssd1.3 (SCL); no longer U1.22 (GPIO17)
- net SSD1306-SDA: now also U1.6 (GPIO4), ssd1.4 (SDA); no longer U1.21 (GPIO16)
- net VCC: now also ssd1.2 (VCC)
- net at MX7.2 (ROW): now also D6.A
- net at MX6.2 (ROW): now also D5.A
- net at MX2.2 (ROW): now also D1.A
- net at MX9.2 (ROW): now also D8.A
- net at MX8.2 (ROW): now also D7.A
- net at MX1.2 (ROW): now also D10.A
- net at MX5.2 (ROW): now also D4.A
- net at MX3.2 (ROW): now also D2.A
- net at MX4.2 (ROW): now also D3.A
