File: 3D4E Macropad.kicad_pcb (KiCad board)
At the start: 2 copper layers, 21 parts, among them U1 Pico, U2 KY-040

Commit message: macropad update final
Parts:
- removed D9: D_Small, Diode_SMD:D_SOD-123
- removed REF**: SSD1306-0.91-OLED-4pin-128x32, KiCad-SSD1306-0.91-OLED-4pin-128x32.pretty-master:SSD1306-0.91-OLED-4pin-128x32
- added ?: LOGO, LOGO, F.Cu at (107.5, 115.0)
- added D0: 1N4148, 1N4148-Diode:DIOAD829W49L456D191, F.Cu at (42.5, 84.4)
- added HOLE_M3: VAL**, keyboard_parts.pretty-master:HOLE_M3, F.Cu at (25.0, 125.0)
- added HOLE_M3: VAL**, keyboard_parts.pretty-master:HOLE_M3, F.Cu at (25.0, 70.0)
- added HOLE_M3: VAL**, keyboard_parts.pretty-master:HOLE_M3, F.Cu at (120.0, 125.0)
- added ssd1: 3, KiCad-SSD1306-0.91-OLED-4pin-128x32.pretty-master:SSD1306-0.91-OLED-4pin-128x32, F.Cu at (55.0, 52.8)
- D1, D2, D3, D4, D5, D6, D7, D8: value D_Small -> 1N4148; footprint Diode_SMD:D_SOD-123 -> 1N4148-Diode:DIOAD829W49L456D191
- moved U2 152.0 mm to (27.5, 59.8)
- moved MX7 131.4 mm to (42.4, 114.3)
- moved D7 112.6 mm to (61.4, 122.5)
- moved MX8 110.1 mm to (61.5, 114.3)
- moved D6 107.5 mm to (42.4, 122.5)
- moved MX4 103.9 mm to (42.4, 95.2)
- moved MX9 95.3 mm to (80.5, 114.3)
- moved D8 90.8 mm to (80.6, 122.5)
- moved D3 90.7 mm to (42.5, 103.5)
- moved MX5 87.2 mm to (61.5, 95.2)
- moved D4 84.7 mm to (61.5, 103.5)
- moved MX6 80.8 mm to (80.5, 95.2)
- moved MX1 78.7 mm to (42.4, 76.2)
- moved MX3 77.0 mm to (80.5, 76.2)
- moved MX2 70.8 mm to (61.4, 76.2)
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Connections:
- MX1 pad 2: Net-(D1-A) -> Net-(MX1-ROW)
- MX2 pad 2: Net-(D2-A) -> Net-(MX2-ROW)
- MX3 pad 2: Net-(D3-A) -> Net-(MX3-ROW)
- MX4 pad 2: Net-(D4-A) -> Net-(MX4-ROW)
- MX5 pad 2: Net-(D5-A) -> Net-(MX5-ROW)
- MX6 pad 2: Net-(D6-A) -> Net-(MX6-ROW)
- MX7 pad 2: Net-(D7-A) -> Net-(MX7-ROW)
- MX8 pad 2: Net-(D8-A) -> Net-(MX8-ROW)
- MX9 pad 2: Net-(D9-A) -> Net-(MX9-ROW)
- U1 pad 1: unconnected-(U1-GPIO0-Pad1) -> KY040-CLK
- U1 pad 10: unconnected-(U1-GPIO7-Pad10) -> Col 1
- U1 pad 11: unconnected-(U1-GPIO8-Pad11) -> Col 2
- U1 pad 12: Row_0 -> unconnected-(U1-GPIO9-Pad12)
- U1 pad 13: Row_1 -> GND
- U1 pad 17: unconnected-(U1-GPIO13-Pad17) -> Row_0
- U1 pad 18: unconnected-(U1-GND-Pad18) -> GND
- U1 pad 19: unconnected-(U1-GPIO14-Pad19) -> Row_1
- U1 pad 2: unconnected-(U1-GPIO1-Pad2) -> KY040-DT
- U1 pad 20: unconnected-(U1-GPIO15-Pad20) -> Row_2
- U1 pad 21: SSD1306-SDA -> unconnected-(U1-GPIO16-Pad21)
- U1 pad 22: SSD1306-SCK -> unconnected-(U1-GPIO17-Pad22)
- U1 pad 29: Row_2 -> unconnected-(U1-GPIO22-Pad29)
- U1 pad 31: KY040-CLK -> unconnected-(U1-GPIO26_ADC0-Pad31)
- U1 pad 32: KY040-DT -> unconnected-(U1-GPIO27_ADC1-Pad32)
- U1 pad 34: KY040-SW -> unconnected-(U1-GPIO28_ADC2-Pad34)
- U1 pad 4: Col 2 -> KY040-SW
- U1 pad 5: Col 1 -> unconnected-(U1-GPIO3-Pad5)
- U1 pad 6: Col 0 -> SSD1306-SDA
- U1 pad 7: unconnected-(U1-GPIO5-Pad7) -> SSD1306-SCK
- U1 pad 8: unconnected-(U1-GND-Pad8) -> GND
- U1 pad 9: unconnected-(U1-GPIO6-Pad9) -> Col 0
Routing:
- net VCC: track 24.4 -> 108.9 mm
- net Col 2: track 144.6 -> 72.5 mm
- net GND: track 27.6 -> 80.3 mm
- net KY040-SW: track 32.6 -> 70.5 mm
- net KY040-CLK: track 41.1 -> 71.0 mm
- net Col 0: track 86.3 -> 112.5 mm
- net Row_1: track 84.8 -> 63.7 mm
- net Col 1: track 113.9 -> 92.9 mm
- net Net-(MX2-ROW): track 0.00 -> 19.9 mm
- net Net-(MX3-ROW): track 0.00 -> 19.8 mm
- net Net-(MX7-ROW): track 0.00 -> 19.8 mm
- net Net-(MX4-ROW): track 0.00 -> 19.7 mm
- net Net-(MX8-ROW): track 0.00 -> 19.4 mm
- net Net-(MX1-ROW): track 0.00 -> 19.4 mm
- net Net-(MX6-ROW): track 0.00 -> 19.4 mm
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
Commit message: fixed positioning of rotary encoder pcb
Parts:
- moved U2 20.1 mm to (47.5, 57.9)
Routing:
- net KY040-DT: track 71.9 -> 52.7 mm
- net VCC: track 108.9 -> 89.7 mm
- net KY040-CLK: track 71.0 -> 51.9 mm
- net GND: track 80.3 -> 61.2 mm
- net KY040-SW: track 70.5 -> 51.6 mm
Changed lines of the file:
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@@
   )
   (footprint "KY-040:KY-040-PORT" (layer "F.Cu")
-    (at 27.5 59.77 -90)
+    (at 47.5 57.93 -90)
     (descr "<b>PIN HEADER</b>")
     (property "Availability" "Not in stock")
@@
   (segment (start 71 122.5) (end 71 123.5) (width 0.381) (layer "B.Cu") (net 6))
   (segment (start 84.792 119.208) (end 89.5 114.5) (width 0.381) (layer "B.Cu") (net 6))
+  (segment (start 95 56.5) (end 97.64 56.5) (width 0.381) (layer "B.Cu") (net 23))
+  (segment (start 91.5 55) (end 93.5 55) (width 0.381) (layer "B.Cu") (net 23))
+  (segment (start 48.58 61.74) (end 50.42 63.58) (width 0.381) (layer "B.Cu") (net 23))
+  (segment (start 97.64 56.5) (end 97.72 56.58) (width 0.381) (layer "B.Cu") (net 23))
+  (segment (start 97.44 69) (end 97.72 69.28) (width 0.381) (layer "B.Cu") (net 23))
+  (segment (start 47.5 61.74) (end 48.58 61.74) (width 0.381) (layer "B.Cu") (net 23))
+  (segment (start 87.5 65.5) (end 92.5 65.5) (width 0.381) (layer "B.Cu") (net 23))
+  (segment (start 50.42 63.58) (end 85.58 63.58) (width 0.381) (layer "B.Cu") (net 23))
+  (segment (start 93.5 68) (end 94.5 69) (width 0.381) (layer "B.Cu") (net 23))
+  (segment (start 92.5 65.5) (end 93.5 66.5) (width 0.381) (layer "B.Cu") (net 23))
   (segment (start 93.5 66.5) (end 93.5 68) (width 0.381) (layer "B.Cu") (net 23))
-  (segment (start 95 56.5) (end 97.64 56.5) (width 0.381) (layer "B.Cu") (net 23))
-  (segment (start 27.5 63.58) (end 85.58 63.58) (width 0.381) (layer "B.Cu") (net 23))
-  (segment (start 91.5 55) (end 93.5 55) (width 0.381) (layer "B.Cu") (net 23))
+  (segment (start 47.5 61.74) (end 47.58 61.66) (width 0.381) (layer "B.Cu") (net 23))
+  (segment (start 94.5 69) (end 97.44 69) (width 0.381) (layer "B.Cu") (net 23))
   (segment (start 85.58 63.58) (end 87.5 65.5) (width 0.381) (layer "B.Cu") (net 23))
-  (segment (start 93.5 68) (end 94.5 69) (width 0.381) (layer "B.Cu") (net 23))
-  (segment (start 97.64 56.5) (end 97.72 56.58) (width 0.381) (layer "B.Cu") (net 23))
-  (segment (start 87.5 65.5) (end 92.5 65.5) (width 0.381) (layer "B.Cu") (net 23))
-  (segment (start 94.5 69) (end 97.44 69) (width 0.381) (layer "B.Cu") (net 23))
-  (segment (start 97.44 69) (end 97.72 69.28) (width 0.381) (layer "B.Cu") (net 23))
   (segment (start 93.5 55) (end 95 56.5) (width 0.381) (layer "B.Cu") (net 23))
-  (segment (start 92.5 65.5) (end 93.5 66.5) (width 0.381) (layer "B.Cu") (net 23))
-  (segment (start 27.5 58.5) (end 27.844156 58.844156) (width 0.381) (layer "F.Cu") (net 24))
-  (segment (start 27.844156 58.844156) (end 97.444156 58.844156) (width 0.381) (layer "F.Cu") (net 24))
   (segment (start 97.444156 58.844156) (end 97.72 59.12) (width 0.381) (layer "F.Cu") (net 24))
+  (segment (start 47.5 56.66) (end 47.764156 56.924156) (width 0.381) (layer "F.Cu") (net 24))
+  (segment (start 48.58 56.66) (end 50.764156 58.844156) (width 0.381) (layer "F.Cu") (net 24))
+  (segment (start 50.764156 58.844156) (end 97.444156 58.844156) (width 0.381) (layer "F.Cu") (net 24))
+  (segment (start 47.5 56.66) (end 48.58 56.66) (width 0.381) (layer "F.Cu") (net 24))
+  (segment (start 94 53) (end 95.04 54.04) (width 0.381) (layer "F.Cu") (net 25))
+  (segment (start 47.5 54.12) (end 48.58 54.12) (width 0.381) (layer "F.Cu") (net 25))
+  (segment (start 48.58 54.12) (end 50.46 56) (width 0.381) (layer "F.Cu") (net 25))
+  (segment (start 47.5 54.12) (end 47.54 54.08) (width 0.381) (layer "F.Cu") (net 25))
+  (segment (start 50.46 56) (end 85.5 56) (width 0.381) (layer "F.Cu") (net 25))
+  (segment (start 88.5 53) (end 94 53) (width 0.381) (layer "F.Cu") (net 25))
+  (segment (start 85.5 56) (end 88.5 53) (width 0.381) (layer "F.Cu") (net 25))
   (segment (start 95.04 54.04) (end 97.72 54.04) (width 0.381) (layer "F.Cu") (net 25))
-  (segment (start 88.5 53) (end 94 53) (width 0.381) (layer "F.Cu") (net 25))
-  (segment (start 85.54 55.96) (end 88.5 53) (width 0.381) (layer "F.Cu") (net 25))
-  (segment (start 94 53) (end 95.04 54.04) (width 0.381) (layer "F.Cu") (net 25))
-  (segment (start 27.5 55.96) (end 85.54 55.96) (width 0.381) (layer "F.Cu") (net 25))
-  (segment (start 27.5 53.42) (end 86.08 53.42) (width 0.381) (layer "F.Cu") (net 26))
   (segment (start 86.08 53.42) (end 88 51.5) (width 0.381) (layer "F.Cu") (net 26))
+  (segment (start 50.42 53.42) (end 86.08 53.42) (width 0.381) (layer "F.Cu") (net 26))
   (segment (start 88 51.5) (end 97.72 51.5) (width 0.381) (layer "F.Cu") (net 26))
+  (segment (start 47.5 51.58) (end 47.58 51.5) (width 0.381) (layer "F.Cu") (net 26))
+  (segment (start 47.5 51.58) (end 48.58 51.58) (width 0.381) (layer "F.Cu") (net 26))
+  (segment (start 48.58 51.58) (end 50.42 53.42) (width 0.381) (layer "F.Cu") (net 26))
+  (segment (start 47.5 59.2) (end 47.58 59.12) (width 0.381) (layer "B.Cu") (net 31))
+  (segment (start 48.58 59.2) (end 50.42 61.04) (width 0.381) (layer "B.Cu") (net 31))
   (segment (start 94.5 64.5) (end 94.5 63) (width 0.381) (layer "B.Cu") (net 31))
+  (segment (start 105.855844 62.964156) (end 107.16 61.66) (width 0.381) (layer "B.Cu") (net 31))
+  (segment (start 91.5 57.54) (end 91.844156 57.884156) (width 0.381) (layer "B.Cu") (net 31))
+  (segment (start 47.5 59.2) (end 48.58 59.2) (width 0.381) (layer "B.Cu") (net 31))
   (segment (start 86.54 61.04) (end 90 64.5) (width 0.381) (layer "B.Cu") (net 31))
-  (segment (start 91.5 57.54) (end 91.844156 57.884156) (width 0.381) (layer "B.Cu") (net 31))
+  (segment (start 90 64.5) (end 94.5 64.5) (width 0.381) (layer "B.Cu") (net 31))
+  (segment (start 107.16 61.66) (end 115.5 61.66) (width 0.381) (layer "B.Cu") (net 31))
   (segment (start 94.535844 62.964156) (end 105.855844 62.964156) (width 0.381) (layer "B.Cu") (net 31))
-  (segment (start 107.16 61.66) (end 115.5 61.66) (width 0.381) (layer "B.Cu") (net 31))
-  (segment (start 90 64.5) (end 94.5 64.5) (width 0.381) (layer "B.Cu") (net 31))
+  (segment (start 91.844156 57.884156) (end 103.384156 57.884156) (width 0.381) (layer "B.Cu") (net 31))
   (segment (start 94.5 63) (end 94.535844 62.964156) (width 0.381) (layer "B.Cu") (net 31))
-  (segment (start 91.844156 57.884156) (end 103.384156 57.884156) (width 0.381) (layer "B.Cu") (net 31))
-  (segment (start 105.855844 62.964156) (end 107.16 61.66) (width 0.381) (layer "B.Cu") (net 31))
   (segment (start 103.384156 57.884156) (end 107.16 61.66) (width 0.381) (layer "B.Cu") (net 31))
-  (segment (start 27.5 61.04) (end 86.54 61.04) (width 0.381) (layer "B.Cu") (net 31))
+  (segment (start 50.42 61.04) (end 86.54 61.04) (width 0.381) (layer "B.Cu") (net 31))
   (segment (start 93.5 66.5) (end 97.48 66.5) (width 0.381) (layer "F.Cu") (net 32))
   (segment (start 90 65.5) (end 92.5 65.5) (width 0.381) (layer "F.Cu") (net 32))

Commit message: bongo cat svg
Parts:
- removed ?: LOGO, LOGO
- added G***: LOGO, LOGO, F.Cu at (105.4, 112.8)

Commit message: flowerpot svg
Parts:
- moved G*** 1.30 mm to (106.5, 113.5)
