File: 3D4E Macropad.kicad_pcb (KiCad board)
At the start: 2 copper layers, 25 parts, among them U1 Pico, U2 KY-040

Commit message: update to graphics
Parts:
- removed ?: LOGO, LOGO
- added G***: LOGO, LOGO, F.Cu at (106.5, 114.5)
